File: device/*/_autosave-*.kicad_pcb (KiCad board)
At the start: 2 copper layers, 99.5 x 99.5 mm, 7 parts, among them SW1 SW_Push, SW2 SW_Push

Commit message: feat: server send local time back
Connections:
- DS2 pad 1: GND -> Net-(DS2-LED(-))
- DS2 pad 16: GND -> Net-(DS2-LED(-))
- DS2 pad 5: GND -> Net-(DS2-LED(-))
- Esp32-Wroom-32D1 pad 1: GND -> Net-(Esp32-Wroom-32D1-GND-Pad1)
- Esp32-Wroom-32D1 pad 38: GND -> Net-(DS2-LED(-))
- R2 pad 2: GND -> Net-(Esp32-Wroom-32D1-GND-Pad1)
- R3 pad 1: GND -> Net-(DS2-LED(-))
- SW1 pad 2: GND -> Net-(Esp32-Wroom-32D1-GND-Pad1)
- SW2 pad 2: GND -> Net-(Esp32-Wroom-32D1-GND-Pad1)
Routing:
- added copper zone on B.Cu, net Net-(Esp32-Wroom-32D1-GND-Pad1)
- added copper zone on F.Cu, net Net-(Esp32-Wroom-32D1-GND-Pad1)
- removed copper zone on B.Cu, net GND
- removed copper zone on F.Cu, net GND
